Commit message: In this I create a hardware interface yaml that uses the one supplied by the examples in the demo so that now I can write a node that just controls them, this is just awesome

File: description/robot.urdf.xacro (robot description, xacro)
@@ -5,3 +5,4 @@
   <!-- Import Rviz colors -->
   <xacro:include filename="rrbot.materials.xacro"/>
+  <xacro:include filename="rrbot.ros2_control.xacro"/>
 </robot>

File: description/rrbot_description.urdf.xacro (robot description, xacro)
@@ -39,4 +39,7 @@
     </inertial>
   </link>
+    <gazebo reference="base_link">
+        <material>Gazebo/Orange</material>
+    </gazebo>
   <!-- First Joint -->
   <joint name="joint1" type="continuous">
@@ -71,4 +74,7 @@
     </inertial>
   </link>
+    <gazebo reference="link1">
+        <material>Gazebo/White</material>
+    </gazebo>
   <!-- Second Link -->
   <joint name="joint2" type="continuous">
@@ -103,4 +109,7 @@
     </inertial>
   </link>
+    <gazebo reference="link2">
+        <material>Gazebo/Orange</material>
+    </gazebo>
   <joint name="tool_joint" type="fixed">
     <origin xyz="0 0 1" rpy="0 0 0" />
